File: Segment/Segment.kicad_pcb (KiCad board)
At the start: 2 copper layers, 130.2 x 10.2 mm, 17 parts, among them J1 1x03, J2 1x03

Commit message: Added text and logos. Ordered version
Parts:
- added G***: LOGO, Logos:logo_MLlabs_small, B.Cu at (192.3, 105.7)
- added G***: LOGO, Logos:logo_MLlabs_small, B.Cu at (127.8, 105.7)
Other:
- board text added: "APA-106-F8 7-Seg"
