File: Segment/Segment.kicad_pcb (KiCad board)
At the start: 2 copper layers, 130.2 x 10.2 mm, 19 parts, among them J1 1x03, J2 1x03

Commit message: Fix shorts
Routing:
- net +5V: track 215.5 -> 180.3 mm
